File: SDLH.kicad_sch (KiCad schematic)
At the start: 67 parts, among them J1 RST, J2 BSEL, K1 Relay_SPDT_G6RN, K2 Relay_SPDT_G6RN, Q1 BSS205N, Q2 BSS205N, U1 TLV1702, U2 ISO1044BD, U3 CD4043BE, U4 ESP32-S3-WROOM-1U-N4R2, U5 TLV1702, U6 TLV1702, U7 TLV1702

Commit message: Add files via upload
Parts:
- added C8, C9: 10u, symbol Device:C
- added D3, D4: D, symbol Device:D
- added Q3, Q4, Q5, Q6: BSS205N, Custom_MSM:MOSFET_Single_SOT-23, symbol Custom_MSM:MOSFET_N-CH
- added R30, R31: 100k, symbol Device:R
- added R32, R33: 1k, symbol Device:R
- added R34, R35: R, symbol Device:R
- added U8: 74AHC2G00, symbol 74xGxx:74AHC2G00
Connections:
- net +12V: now also K1.5, K2.5, D3.1 (K), D4.1 (K)
- net +5V: now also C8.1, C9.1
- net AMS_Latch: now also U8.5, U8.6
- net GND: now also Q3.2 (S), Q4.2 (S), Q5.2 (S), Q6.2 (S), R30.2, R31.2
- net IMD_Latch: now also U8.1, U8.2
- net Light_AMS: now also R33.1
- net Light_IMD: now also R32.1
- net at K2.1: now also D4.2 (A), Q6.3 (D)
- net at K2.2: now also K1.2
- net SDC_Out: now reaches K2.3
- net at K1.1: now also D3.2 (A), Q5.3 (D)
- net SDC_In: now reaches K1.3
- new net: Q5.1 (G), R34.2
- new net: C9.2, Q4.1 (G), R31.1
- new net: Q6.1 (G), R35.1
- new net: C8.2, Q3.1 (G), R30.1
- new net: Q3.3 (D), R32.2
- new net: Q4.3 (D), R33.2
- new net IAMS_Latch: R34.1, U8.3
- new net IIMD_Latch: R35.2, U8.7
- no-connect marks 41 -> 43
Other:
- note added: "Hold the fault lights on start up"
- note added: "Inverters"
- note added: "Shutdown Relays"
- moved on the sheet: K1, K2, R21, TP4, U7A, U7B
